Commit message: Added marten single leg sources

File: camel-urdf/camel_marten_single_leg/marten_single_leg.urdf (robot description, URDF)
Before this commit: robot JHdog-single-leg, 5 links, 4 joints
Links:
- added link hip_2, mass 0.337
- link hip_1: mass 0.7835 -> 0.337; geometry collision cylinder length=0.04 radius=0.038; visual mesh filename=hip.STL
- link lower_leg: mass 1.0 -> 0.171; geometry collision sphere radius=0.010; visual mesh filename=calf.STL
- link upper_leg: mass 0.221 -> 0.171; geometry collision box size=0.035 0.04 0.18; visual mesh filename=thigh.STL
Joints:
- added joint hip_upper: type fixed, parent hip_2, child upper_leg, origin xyz=0 0 0 rpy=0 0 0
- joint hip_pitch: axis 0 1 0 -> 0 -1 0; child upper_leg -> hip_2
- joint knee_pitch: axis 0 1 0 -> 0 -1 0; origin xyz=0 -0.064 -0.18 rpy=0 0 0 -> xyz=0 -0.065 -0.18 rpy=0 0 0
- joint linear_guide: origin xyz=0 -0.03525 0.0 rpy=0 0 0 -> xyz=0 -0.025 0.0 rpy=0 0 0

Commit message: Updated mass of linear guide

File: camel-urdf/camel_marten_single_leg/marten_single_leg.urdf (robot description, URDF)
Before this commit: robot marten-single-leg, 6 links, 5 joints
Links:
- link hip_1: mass 0.337 -> 1.073
